File: Boards/PulverTech_v1/PulverTech_v1.sch (EAGLE design)
At the start: 40 parts, among them IC1 786TV, K1 G5LE, P1 FSMCD, Q1 16.0 mHz, Q4 BC548, Q6 IRF540, Q7 IRF540, Q8 IRF9530, Q9 IRF9530, U1 ATMEGA328P-PU

Commit message: final project updates
Parts:
- removed R1, R2, R5, R6: 10k, eagle-ltspice:R0204/7
- removed X1: (no value), con-ptr500:AK500/2
- added C3: 100nF, capacitor-wima:C2.5/2
- added D2, D3: 1N4733, diode:1N4728
- added D5, D6, D7: 1N4007, diode:1N4004
- added POWER: (no value), con-ptr500:AK500/2
- R16, R4: value 10k -> 30k
- renumbered P1 to RESET, X2 to VALVE, X3 to SECTION, X4 to SPEED, X5 to FLUX
Connections:
- removed net N$31: R4.1, R5.1
- net GND: now also D1.A, D2.A, D3.A, D7.A; no longer R2.1, R6.1, X1-2.KL
- net MOTOR_A: now also C3.2
- net MOTOR_B: now also C3.1
- net N$4: now also D1.C, D5.A, POWER-1.KL; no longer R1.2, R16.1
- net N$5: now also D6.A, D7.C, POWER-2.KL; no longer D1.A, X1-1.KL
- net SENSOR_FLUX: now also D2.C, R16.1; no longer R1.1, R2.2
- net SENSOR_IND: now also D3.C, R4.1; no longer R5.2, R6.2
- net VIN: now also D5.C, D6.C; no longer D1.C
Other:
- moved on the sheet: C1, C2, C4, C5, D1, IC1, LED1, Q1, R16, R3, U1
